File: electronics/spectrum_analyzer_display/spectrum_analyzer_display.kicad_pcb (KiCad board)
At the start: 2 copper layers, 99.1 x 66 mm, 20 parts, among them J1 Conn_01x10_Pin, J2 Conn_01x14_Pin

Commit message: chore: remove files
Changed lines of the file:
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@@
     (effects (font (size 1 1) (thickness 0.15)))
   )
-  (gr_text "R4" (at 111.76 93.98) (layer "F.SilkS")
+  (gr_text "R6" (at 111.76 93.98) (layer "F.SilkS")
     (effects (font (size 1 1) (thickness 0.15)))
   )
@@
     (effects (font (size 1 1) (thickness 0.15)))
   )
-  (gr_text "L4" (at 93.98 93.98) (layer "F.SilkS")
+  (gr_text "L2" (at 93.98 93.98) (layer "F.SilkS")
     (effects (font (size 1 1) (thickness 0.15)))
   )
@@
     (effects (font (size 1 1) (thickness 0.15)))
   )
-  (gr_text "L7" (at 101.6 93.98) (layer "F.SilkS")
+  (gr_text "R4" (at 101.6 93.98) (layer "F.SilkS")
     (effects (font (size 1 1) (thickness 0.15)))
   )
@@
     (effects (font (size 1 1) (thickness 0.15)))
   )
-  (gr_text "R3" (at 109.22 93.98) (layer "F.SilkS")
+  (gr_text "L5" (at 109.22 93.98) (layer "F.SilkS")
     (effects (font (size 1 1) (thickness 0.15)))
   )
-  (gr_text "R2" (at 106.68 93.98) (layer "F.SilkS")
+  (gr_text "R5" (at 106.68 93.98) (layer "F.SilkS")
     (effects (font (size 1 1) (thickness 0.15)))
   )
@@
     (effects (font (size 1 1) (thickness 0.15)))
   )
-  (gr_text "R1" (at 104.14 93.98) (layer "F.SilkS")
+  (gr_text "L4" (at 104.14 93.98) (layer "F.SilkS")
     (effects (font (size 1 1) (thickness 0.15)))
   )
@@
     (effects (font (size 1 1) (thickness 0.15)))
   )
-  (gr_text "L5" (at 96.52 93.98) (layer "F.SilkS")
+  (gr_text "R3" (at 96.52 93.98) (layer "F.SilkS")
     (effects (font (size 1 1) (thickness 0.15)))
   )
@@
     (effects (font (size 1 1) (thickness 0.15)))
   )
-  (gr_text "L2" (at 88.9 93.98) (layer "F.SilkS")
+  (gr_text "R1" (at 88.9 93.98) (layer "F.SilkS")
     (effects (font (size 1 1) (thickness 0.15)))
   )
@@
     (effects (font (size 1 1) (thickness 0.15)))
   )
-  (gr_text "L3" (at 91.44 93.98) (layer "F.SilkS")
+  (gr_text "R2" (at 91.44 93.98) (layer "F.SilkS")
     (effects (font (size 1 1) (thickness 0.15)))
   )
-  (gr_text "R5" (at 114.3 93.98) (layer "F.SilkS")
+  (gr_text "L6" (at 114.3 93.98) (layer "F.SilkS")
     (effects (font (size 1 1) (thickness 0.15)))
   )
@@
     (effects (font (size 1 1) (thickness 0.15)))
   )
-  (gr_text "R6" (at 116.84 93.98) (layer "F.SilkS")
+  (gr_text "L7" (at 116.84 93.98) (layer "F.SilkS")
     (effects (font (size 1 1) (thickness 0.15)))
   )
-  (gr_text "L6" (at 99.06 93.98) (layer "F.SilkS")
+  (gr_text "L3" (at 99.06 93.98) (layer "F.SilkS")
     (effects (font (size 1 1) (thickness 0.15)))
   )
